File: src/kicad-vero/mosfet_double_buffer.kicad_pcb (KiCad board)
At the start: 2 copper layers, 22.9 x 43.2 mm, 24 parts, among them P1 InA, P2 OutA, P3 CONN_2, P3 InB, P4 CONN_2, P4 OutB, P5 Power, Q1 BS170, Q2 BS170

Commit message: finalisation
Other:
- board text added: "Higth 16"
- board text added: "Width 8"
